File: kicad/Flash.kicad_sch (KiCad schematic)
At the start: 35 parts, among them J17 5077CR-16-SMC2-BK-TR, J18 COM, J19 Charge1, J20 Charge2, Q11 BSS138, Q12 BSS138, SW3 ENABLE, SW4 BOOT, U10 NJM2863F33, U11 CH340K, U12 MCP73831-2-OT, U13 MCP73831-2-OT, U14 MCP73831-2-OT

Commit message: とりあえず配線完了
Connections:
- net GND: now also SW3.1 (A); no longer SW3.3 (C)
- net VBUS_FUSE: now reaches F1.1, J17.A4 (VBUS), J17.A9 (VBUS), J17.B4 (VBUS), J17.B9 (VBUS)
Other:
- moved on the sheet: F1
Changed lines of the file:
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@@
   (no_connect (at 64.77 123.19))
   (no_connect (at 64.77 125.73))
-  (no_connect (at 100.33 60.96))
+  (no_connect (at 100.33 66.04))
   (no_connect (at 133.35 109.22))
   (no_connect (at 130.81 149.86))
@@
     (stroke (width 0) (type default))
   )
-  (wire (pts (xy 74.93 95.25) (xy 77.47 95.25))
+  (wire (pts (xy 82.55 95.25) (xy 85.09 95.25))
     (stroke (width 0) (type default))
   )
@@
     (stroke (width 0) (type default))
   )
-  (wire (pts (xy 64.77 95.25) (xy 67.31 95.25))
+  (wire (pts (xy 64.77 95.25) (xy 74.93 95.25))
     (stroke (width 0) (type default))
   )
@@
     (effects (font (size 1.27 1.27)) (justify right bottom))
   )
-  (label "GND" (at 100.33 66.04 0) (fields_autoplaced)
+  (label "GND" (at 100.33 60.96 0) (fields_autoplaced)
     (effects (font (size 1.27 1.27)) (justify left bottom))
   )
@@
     (effects (font (size 1.27 1.27)) (justify right bottom))
   )
-  (label "VBUS" (at 77.47 95.25 0) (fields_autoplaced)
+  (label "VBUS" (at 85.09 95.25 0) (fields_autoplaced)
     (effects (font (size 1.27 1.27)) (justify left bottom))
   )
@@
   (label "GND" (at 123.19 129.54 180) (fields_autoplaced)
     (effects (font (size 1.27 1.27)) (justify right bottom))
+  )
+  (label "VBUS_FUSE" (at 64.77 95.25 0) (fields_autoplaced)
+    (effects (font (size 1.27 1.27)) (justify left bottom))
   )
   (label "USB_D-" (at 64.77 107.95 0) (fields_autoplaced)
@@
     )
   )
-  (symbol (lib_id "Device:Polyfuse") (at 71.12 95.25 90) (unit 1)
+  (symbol (lib_id "Device:Polyfuse") (at 78.74 95.25 90) (unit 1)
     (in_bom yes) (on_board yes) (dnp no)
-    (property "Reference" "F1" (at 71.12 90.17 90)
+    (property "Reference" "F1" (at 78.74 90.17 90)
       (effects (font (size 1.27 1.27)))
     )
-    (property "Value" "MF-FSMF035X-2" (at 71.12 92.71 90)
+    (property "Value" "MF-FSMF035X-2" (at 78.74 92.71 90)
       (effects (font (size 1.27 1.27)))
     )
-    (property "Footprint" "Resistor_SMD:R_0603_1608Metric" (at 76.2 93.98 0)
+    (property "Footprint" "Resistor_SMD:R_0603_1608Metric" (at 83.82 93.98 0)
       (effects (font (size 1.27 1.27)) (justify left) hide)
     )
-    (property "Datasheet" "~" (at 71.12 95.25 0)
-      (effects (font (size 1.27 1.27)) hide)
-    )
+    (property "Datasheet" "~" (at 78.74 95.25 0)
+      (effects (font (size 1.27 1.27)) hide)
+    )

Commit message: 1回目の基板修正
Parts:
- removed C29: 1u, Capacitor_SMD:C_0402_1005Metric, symbol Device:C_Small
- removed Q11, Q12: BSS138, Package_TO_SOT_SMD:SOT-23, symbol Transistor_FET:BSS138
- removed SW3: ENABLE, Button_Switch_SMD:SW_SPDT_PCM12, symbol Switch:SW_SPDT
- removed U11: CH340K, Package_SO:SSOP-10_3.9x4.9mm_P1.00mm, symbol KERISE:CH340K
- added SW3: RESET, Button_Switch_SMD:SW_Push_1P1T_NO_Vertical_Wuerth_434133025816, symbol Switch:SW_Push
- added U10: FT234XD, Package_DFN_QFN:DFN-12-1EP_3x3mm_P0.5mm_EP1.6x2.5mm, symbol KERISE:FT234XD
- R19, R20, R21: value 4.7k -> 1k
- renumbered C30 to C29, C31 to C30, C32 to C31, C33 to C32, C34 to C33, C35 to C34, J18 to J17, J17 to J18, U10 to U11
Connections:
- net ESP32_EN: now also SW3.1
- net ESP32_RX: now also U10.7 (TXD)
- net ESP32_TX: now also U10.10 (RXD)
- net GND: now also SW3.2, U10.13 (GND), U10.5 (GND)
- net USB_D+: now also U10.12 (USBDP)
- net USB_D-: now also U10.1 (USBDM)
- net VCC: now also C26.2, U10.2 (RESET#), U10.3 (3V3OUT), U10.4 (VCC), U10.9 (VCCIO)
- no-connect marks 5 -> 6
Other:
- moved on the sheet: C26, C27, C28, J17, SW4, U11
