File: kicad/IR_RCV.kicad_sch (KiCad schematic)
At the start: 9 parts, among them J11 Ref_Host, J12 Ref_Slave, Q6 DMN3065LW-7, Q7 APDA3020P3C-P22

Commit message: 1回目の基板修正
Parts:
- R7: footprint Resistor_SMD:R_0603_1608Metric -> Resistor_SMD:R_0402_1005Metric
Changed lines of the file:
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@@
       (effects (font (size 1.27 1.27)))
     )
-    (property "Footprint" "Resistor_SMD:R_0603_1608Metric" (at 111.252 99.06 90)
+    (property "Footprint" "Resistor_SMD:R_0402_1005Metric" (at 111.252 99.06 90)
       (effects (font (size 1.27 1.27)) hide)
     )
